File: Commander-Board.sch (KiCad schematic (older format))
At the start: 19 parts

Commit message: Connections between devices.
Parts:
- added C? (x5): C, symbol Device:C
- added J? (x3): Conn_01x04_Female, symbol Connector:Conn_01x04_Female
- added R? (x2): R, symbol Device:R
- TP?: value PROG_GND -> SERVICE_GND
- TP?: value PROG_3V3 -> SERVICE_3V3
- TP?: value PROG_RX -> SERVICE_RX
- TP?: value PROG_TX -> SERVICE_TX
- TP?: value PROG_BOOT -> SERVICE_BOOT
Connections:
- net labels added: ENC_A, ENC_B, PB_BACK, PB_ENT, PR_BOOT, PR_RX, PR_TX, SPI_TFT, TFT_BL, TFT_CS, TFT_DI, TFT_RS, TFT_RST, TFT_SCK, UART_SERVICE
- wire segments 57 -> 76
Other:
- moved on the sheet: C?, J?, JP?, R?, SW?, TP?, U?

Commit message: First schematic
Parts:
- removed C? (x3): C, symbol Device:C
- removed J? (x3): Conn_01x04_Female, symbol Connector:Conn_01x04_Female
- removed M?: 3.5_TFT_SPI_480_320, symbol ILI9488_Display:3.5_TFT_SPI_480_320
- removed R?: R, symbol Device:R
- added C1: 100u, symbol Device:CP
- added C6: 220u, symbol Device:CP
- added J?: EXPAND, symbol Connector_Generic:Conn_01x05
- added M1: 3.5_TFT_SPI_480_320, ILI9488_Display:3.5_TFT_SPI_480_320, symbol ILI9488_Display:3.5_TFT_SPI_480_320
- added R?: 10k, symbol Device:R
- added R?: 1k, symbol Device:R
- C3: renamed from C?; value C -> 1u
- C4, C9: renamed from C?; value C -> 100n
- C5: renamed from C?; value C -> 2.2u
- JP1: renamed from JP?; value CS_BYPASS -> BYPASS
- R1: renamed from R?; value LIGHT_SENSOR -> LDR
- R2: renamed from R?; value R -> 1k
- R3: renamed from R?; value R -> 10k
- TP1, TP2, TP3, TP4, TP5: renamed from TP?; footprint (none) -> TestPoint:TestPoint_Pad_D1.5mm
- gave numbers to parts that had none: 8
Connections:
- net +12V: now also C1.1
- net +3V3: now also C4.1, C8.1, R2.2, R3.1, C6.1, J?.1 (Pin_1), M1.13 (GND)
- net GND: now also C4.2, C8.2, C9.1, R1.2, C1.2, C6.2, J?.5 (Pin_5), M1.14 (VCC), R?.2
- net PB_BACK: now also U3.28 (IO17); no longer U3.9 (IO33)
- net PB_ENT: now also U3.27 (IO16); no longer U3.8 (IO32)
- net TFT_BL: now also M1.7 (LED)
- net TFT_CS: now also M1.12 (CS)
- net TFT_DI: now also M1.9 (SDI)
- net TFT_RS: now also M1.10 (DC/RS)
- net TFT_RST: now also M1.11 (RESET)
- net TFT_SCK: now also M1.8 (SCK)
- net EX_3: now reaches U3.14 (IO12)
- net EX_3: now also J?.4 (Pin_4)
- net SD_CS: now reaches U3.29 (IO5)
- net SD_CS: now also M1.15 (SD_CS)
- net at U3.3 (EN): now also C9.2, R3.2
- net SD_SCK: now reaches U3.30 (IO18)
- net SD_SCK: now also M1.18 (SD_SCK)
- net SD_MISO: now reaches U3.31 (IO19)
- net SD_MISO: now also M1.17 (SD_MISO)
- net EX_1: now reaches U3.33 (IO21)
- net EX_1: now also J?.2 (Pin_2)
- net EX_2: now reaches U3.36 (IO22)
- net EX_2: now also J?.3 (Pin_3)
- net SD_MOSI: now reaches U3.37 (IO23)
- net SD_MOSI: now also M1.16 (SD_MOSI)
- net AN_VOLT: now reaches U3.6 (IO34)
- net AN_VOLT: now also R?.1, R?.2
- net at J1.2 (Pin_2): now also R?.1
- net AN_LIGHT: now reaches R1.1
- net AN_LIGHT: now also R2.1, U3.8 (IO32)
- net AN_CURR: now reaches U2.7 (VIOUT)
- net AN_CURR: now also U3.9 (IO33)
- no-connect marks 5 -> 14
Other:
- moved on the sheet: C3, C4, C5, C8, C9, J1, JP1, R1, R2, R3, SW1, SW2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

Commit message: First board test
Parts:
- C1, C6: footprint (none) -> Capacitor_THT:CP_Radial_D10.0mm_P5.00mm
- C3, C4, C8, C9: footprint (none) -> Capacitor_THT:C_Disc_D4.7mm_W2.5mm_P5.00mm
- C5: footprint (none) -> Capacitor_THT:C_Disc_D7.0mm_W2.5mm_P5.00mm
- J1: footprint (none) -> TerminalBlock_MetzConnect:TerminalBlock_MetzConnect_Type011_RT05503HBWC_1x03_P5.00mm_Horizontal
- J2: renamed from J?; footprint (none) -> Connector_PinSocket_2.54mm:PinSocket_1x05_P2.54mm_Horizontal
- JP1: footprint (none) -> Jumper:SolderJumper-2_P1.3mm_Open_RoundedPad1.0x1.5mm
- R1: footprint (none) -> OptoDevice:R_LDR_5.1x4.3mm_P3.4mm_Vertical
- R2, R3: footprint (none) -> Resistor_THT:R_Axial_DIN0207_L6.3mm_D2.5mm_P10.16mm_Horizontal
- R4, R5: renamed from R?; footprint (none) -> Resistor_THT:R_Axial_DIN0207_L6.3mm_D2.5mm_P10.16mm_Horizontal
- SW1, SW2: footprint (none) -> Button_Switch_THT:SW_PUSH_6mm_H4.3mm
Changed lines of the file:
@@
 F 0 "JP1" H 13650 4650 50  0000 R CNN
 F 1 "BYPASS" H 13650 4600 50  0000 R CNN
-F 2 "" H 13500 4750 50  0001 C CNN
+F 2 "Jumper:SolderJumper-2_P1.3mm_Open_RoundedPad1.0x1.5mm" H 13500 4750 50  0001 C CNN
 F 3 "~" H 13500 4750 50  0001 C CNN
 	1    13500 4750
@@
 F 0 "SW1" V 1953 9174 50  0000 C CNN
 F 1 "BUTTON_BACK" V 2050 9350 50  0000 C CNN
-F 2 "" H 2000 9150 50  0001 C CNN
+F 2 "Button_Switch_THT:SW_PUSH_6mm_H4.3mm" H 2000 9150 50  0001 C CNN
 F 3 "~" H 2000 9150 50  0001 C CNN
 	1    2000 8950
@@
 F 0 "J1" H 12368 5167 50  0000 C CNN
 F 1 "POWER" H 12368 5076 50  0000 C CNN
-F 2 "" H 12450 4850 50  0001 C CNN
+F 2 "TerminalBlock_MetzConnect:TerminalBlock_MetzConnect_Type011_RT05503HBWC_1x03_P5.00mm_Horizontal" H 12450 4850 50  0001 C CNN
 F 3 "~" H 12450 4850 50  0001 C CNN
 	1    12450 4850
@@
 F 0 "R1" H 2270 5946 50  0000 L CNN
 F 1 "LDR" H 2270 5855 50  0000 L CNN
-F 2 "" V 2250 5650 50  0001 L CNN
+F 2 "OptoDevice:R_LDR_5.1x4.3mm_P3.4mm_Vertical" V 2250 5650 50  0001 L CNN
 F 3 "~" H 2200 5850 50  0001 C CNN
 	1    2200 5900
@@
 F 0 "SW2" V 1950 9750 50  0000 C CNN
 F 1 "BUTTON_ENTER" V 2050 9950 50  0000 C CNN
-F 2 "" H 2000 9750 50  0001 C CNN
+F 2 "Button_Switch_THT:SW_PUSH_6mm_H4.3mm" H 2000 9750 50  0001 C CNN
 F 3 "~" H 2000 9750 50  0001 C CNN
 	1    2000 9550
@@
 F 0 "C8" H 7815 3196 50  0000 L CNN
 F 1 "C" H 7815 3105 50  0000 L CNN
-F 2 "" H 7738 3000 50  0001 C CNN
+F 2 "Capacitor_THT:C_Disc_D4.7mm_W2.5mm_P5.00mm" H 7738 3000 50  0001 C CNN
 F 3 "~" H 7700 3150 50  0001 C CNN
 	1    7700 3150
@@
 F 0 "C5" H 2965 2096 50  0000 L CNN
 F 1 "2.2u" H 2965 2005 50  0000 L CNN
-F 2 "" H 2888 1900 50  0001 C CNN
+F 2 "Capacitor_THT:C_Disc_D7.0mm_W2.5mm_P5.00mm" H 2888 1900 50  0001 C CNN
 F 3 "~" H 2850 2050 50  0001 C CNN
 	1    2850 2050
@@
 F 0 "C3" H 1965 2096 50  0000 L CNN
 F 1 "1u" H 1965 2005 50  0000 L CNN
-F 2 "" H 1888 1900 50  0001 C CNN
+F 2 "Capacitor_THT:C_Disc_D4.7mm_W2.5mm_P5.00mm" H 1888 1900 50  0001 C CNN
 F 3 "~" H 1850 2050 50  0001 C CNN
 	1    1850 2050
@@
 F 0 "C9" H 8600 3750 50  0000 L CNN
 F 1 "100n" H 8550 3650 50  0000 L CNN
-F 2 "" H 8888 3550 50  0001 C CNN
+F 2 "Capacitor_THT:C_Disc_D4.7mm_W2.5mm_P5.00mm" H 8888 3550 50  0001 C CNN
 F 3 "~" H 8850 3700 50  0001 C CNN
 	1    8850 3700
@@
 F 0 "C4" H 12800 4400 50  0000 L CNN
 F 1 "100n" H 12700 4300 50  0000 L CNN
-F 2 "" H 13038 4200 50  0001 C CNN
+F 2 "Capacitor_THT:C_Disc_D4.7mm_W2.5mm_P5.00mm" H 13038 4200 50  0001 C CNN
 F 3 "~" H 13000 4350 50  0001 C CNN
 	1    13000 4350
@@
 F 0 "R2" H 2100 5450 50  0000 C CNN
 F 1 "1k" H 2100 5350 50  0000 C CNN
-F 2 "" V 2130 5400 50  0001 C CNN
+F 2 "Resistor_THT:R_Axial_DIN0207_L6.3mm_D2.5mm_P10.16mm_Horizontal" V 2130 5400 50  0001 C CNN
 F 3 "~" H 2200 5400 50  0001 C CNN
 	1    2200 5400
@@
 F 0 "C1" H 1300 2100 50  0000 L CNN
 F 1 "100u" H 1200 2000 50  0000 L CNN
-F 2 "" H 1538 1900 50  0001 C CNN
+F 2 "Capacitor_THT:CP_Radial_D10.0mm_P5.00mm" H 1538 1900 50  0001 C CNN
 F 3 "~" H 1500 2050 50  0001 C CNN
 	1    1500 2050
@@
 F 0 "C6" H 3368 2096 50  0000 L CNN
 F 1 "220u" H 3368 2005 50  0000 L CNN
-F 2 "" H 3288 1900 50  0001 C CNN
+F 2 "Capacitor_THT:CP_Radial_D10.0mm_P5.00mm" H 3288 1900 50  0001 C CNN
 F 3 "~" H 3250 2050 50  0001 C CNN
 	1    3250 2050
@@
 	2200 6050 2200 6150
 $Comp
-L power:GND #PWR?
+L power:GND #PWR0118
 U 1 1 5F0D7088
 P 2200 6150
-F 0 "#PWR?" H 2200 5900 50  0001 C CNN
+F 0 "#PWR0118" H 2200 5900 50  0001 C CNN
 F 1 "GND" H 2205 5977 50  0000 C CNN
 F 2 "" H 2200 6150 50  0001 C CNN
@@
 	3250 1700 2850 1700
 $Comp
-L power:GND #PWR?
+L power:GND #PWR0119
 U 1 1 5F13374A
 P 13000 4500
-F 0 "#PWR?" H 13000 4250 50  0001 C CNN
+F 0 "#PWR0119" H 13000 4250 50  0001 C CNN
 F 1 "GND" H 13005 4327 50  0000 C CNN
 F 2 "" H 13000 4500 50  0001 C CNN
@@
 ENCODER
 $Comp
-L Device:R R?
+L Device:R R4
 U 1 1 5F066161
 P 13250 4950
-F 0 "R?" V 13150 4950 50  0000 C CNN
+F 0 "R4" V 13150 4950 50  0000 C CNN
 F 1 "10k" V 13050 4950 50  0000 C CNN
-F 2 "" V 13180 4950 50  0001 C CNN
+F 2 "Resistor_THT:R_Axial_DIN0207_L6.3mm_D2.5mm_P10.16mm_Horizontal" V 13180 4950 50  0001 C CNN
 F 3 "~" H 13250 4950 50  0001 C CNN
 	1    13250 4950
@@
 $EndComp
 $Comp
-L Device:R R?
+L Device:R R5
 U 1 1 5F0667EF
 P 13750 4950
-F 0 "R?" V 13650 4950 50  0000 C CNN
+F 0 "R5" V 13650 4950 50  0000 C CNN
 F 1 "1k" V 13550 4950 50  0000 C CNN
-F 2 "" V 13680 4950 50  0001 C CNN
+F 2 "Resistor_THT:R_Axial_DIN0207_L6.3mm_D2.5mm_P10.16mm_Horizontal" V 13680 4950 50  0001 C CNN
 F 3 "~" H 13750 4950 50  0001 C CNN
 	1    13750 4950
@@
 	13400 4950 13500 4950
 $Comp
-L power:GND #PWR?
+L power:GND #PWR0120
 U 1 1 5F0752E9
 P 14000 5050
-F 0 "#PWR?" H 14000 4800 50  0001 C CNN
+F 0 "#PWR0120" H 14000 4800 50  0001 C CNN
 F 1 "GND" H 14005 4877 50  0000 C CNN
 F 2 "" H 14000 5050 50  0001 C CNN
@@
 AN_VOLT
 $Comp
-L Connector_Generic:Conn_01x05 J?
+L Connector_Generic:Conn_01x05 J2
 U 1 1 5F217DC7
 P 8800 6100
-F 0 "J?" V 8672 6380 50  0000 L CNN
+F 0 "J2" V 8672 6380 50  0000 L CNN
 F 1 "EXPAND" V 8763 6380 50  0000 L CNN
-F 2 "" H 8800 6100 50  0001 C CNN
+F 2 "Connector_PinSocket_2.54mm:PinSocket_1x05_P2.54mm_Horizontal" H 8800 6100 50  0001 C CNN
 F 3 "~" H 8800 6100 50  0001 C CNN
 	1    8800 6100
@@
 	6550 5200 6900 5200
 $Comp
-L power:GND #PWR?
+L power:GND #PWR0121
 U 1 1 5F24CDED
 P 8600 5650
-F 0 "#PWR?" H 8600 5400 50  0001 C CNN
+F 0 "#PWR0121" H 8600 5400 50  0001 C CNN
 F 1 "GND" H 8605 5477 50  0000 C CNN
 F 2 "" H 8600 5650 50  0001 C CNN
@@
 	9000 5650 9000 5900
 $Comp
-L power:+3V3 #PWR?
+L power:+3V3 #PWR0122
 U 1 1 5F24AE52
 P 9000 5650
-F 0 "#PWR?" H 9000 5500 50  0001 C CNN
+F 0 "#PWR0122" H 9000 5500 50  0001 C CNN
 F 1 "+3V3" H 9015 5823 50  0000 C CNN
 F 2 "" H 9000 5650 50  0001 C CNN
@@
 F 0 "R3" H 8500 3950 50  0000 C CNN
 F 1 "10k" H 8750 3950 50  0000 C CNN
-F 2 "" V 8530 3950 50  0001 C CNN
+F 2 "Resistor_THT:R_Axial_DIN0207_L6.3mm_D2.5mm_P10.16mm_Horizontal" V 8530 3950 50  0001 C CNN
 F 3 "~" H 8600 3950 50  0001 C CNN
 	1    8600 3950
@@
 	7500 2950 7500 2850
 $Comp
-L power:GND #PWR?
+L power:GND #PWR0123
 U 1 1 5F2A2BEA
 P 7700 3350
-F 0 "#PWR?" H 7700 3100 50  0001 C CNN
+F 0 "#PWR0123" H 7700 3100 50  0001 C CNN
 F 1 "GND" H 7705 3177 50  0000 C CNN
 F 2 "" H 7700 3350 50  0001 C CNN
@@
 	8600 3700 8700 3700
 $Comp
-L power:GND #PWR?
+L power:GND #PWR0124
 U 1 1 5F2BB532
 P 9100 3700
-F 0 "#PWR?" H 9100 3450 50  0001 C CNN
+F 0 "#PWR0124" H 9100 3450 50  0001 C CNN
 F 1 "GND" H 9105 3527 50  0000 C CNN
 F 2 "" H 9100 3700 50  0001 C CNN
@@
 	8600 4200 8600 4100
 $Comp
-L power:+3V3 #PWR?
+L power:+3V3 #PWR0125
 U 1 1 5F2C16EC
 P 8600 4200
-F 0 "#PWR?" H 8600 4050 50  0001 C CNN
+F 0 "#PWR0125" H 8600 4050 50  0001 C CNN
 F 1 "+3V3" H 8615 4373 50  0000 C CNN
 F 2 "" H 8600 4200 50  0001 C CNN

Commit message: Complete
Parts:
- SW3: footprint (none) -> ILI9488_Display:RotaryEncoder_Alps_EC16B04
Changed lines of the file:
@@
 F 0 "SW3" H 2350 9600 50  0000 L CNN
 F 1 "Rotary_Encoder" H 2350 9500 50  0000 L CNN
-F 2 "" H 2400 9410 50  0001 C CNN
+F 2 "ILI9488_Display:RotaryEncoder_Alps_EC16B04" H 2400 9410 50  0001 C CNN
 F 3 "~" H 2550 9510 50  0001 C CNN
 	1    2550 9250

Commit message: New service connector
Parts:
- M1: symbol ILI9488_Display:3.5_TFT_SPI_480_320 -> Commander-Board-rescue:3.5_TFT_SPI_480_320-ILI9488_Display
- TP1, TP2, TP3, TP4, TP5: footprint TestPoint:TestPoint_Pad_D1.5mm -> TestPoint:TestPoint_Pad_D1.0mm
Changed lines of the file:
@@
 F 0 "TP5" V 7200 9750 50  0000 L CNN
 F 1 "SERVICE_GND" V 7200 9950 50  0000 L CNN
-F 2 "TestPoint:TestPoint_Pad_D1.5mm" H 7400 9550 50  0001 C CNN
+F 2 "TestPoint:TestPoint_Pad_D1.0mm" H 7400 9550 50  0001 C CNN
 F 3 "~" H 7400 9550 50  0001 C CNN
 	1    7200 9550
@@
 F 0 "TP3" V 7200 9550 50  0000 L CNN
 F 1 "SERVICE_RX" V 7200 9750 50  0000 L CNN
-F 2 "TestPoint:TestPoint_Pad_D1.5mm" H 7400 9350 50  0001 C CNN
+F 2 "TestPoint:TestPoint_Pad_D1.0mm" H 7400 9350 50  0001 C CNN
 F 3 "~" H 7400 9350 50  0001 C CNN
 	1    7200 9350
@@
 F 0 "TP2" V 7200 9450 50  0000 L CNN
 F 1 "SERVICE_TX" V 7200 9650 50  0000 L CNN
-F 2 "TestPoint:TestPoint_Pad_D1.5mm" H 7400 9250 50  0001 C CNN
+F 2 "TestPoint:TestPoint_Pad_D1.0mm" H 7400 9250 50  0001 C CNN
 F 3 "~" H 7400 9250 50  0001 C CNN
 	1    7200 9250
@@
 F 0 "TP1" V 7200 9350 50  0000 L CNN
 F 1 "SERVICE_BOOT" V 7200 9550 50  0000 L CNN
-F 2 "TestPoint:TestPoint_Pad_D1.5mm" H 7400 9150 50  0001 C CNN
+F 2 "TestPoint:TestPoint_Pad_D1.0mm" H 7400 9150 50  0001 C CNN
 F 3 "~" H 7400 9150 50  0001 C CNN
 	1    7200 9150
@@
 F 0 "TP4" V 7200 9650 50  0000 L CNN
 F 1 "SERVICE_3V3" V 7200 9850 50  0000 L CNN
-F 2 "TestPoint:TestPoint_Pad_D1.5mm" H 7400 9450 50  0001 C CNN
+F 2 "TestPoint:TestPoint_Pad_D1.0mm" H 7400 9450 50  0001 C CNN
 F 3 "~" H 7400 9450 50  0001 C CNN
 	1    7200 9450
@@
 	12200 9050 14700 9050
 $Comp
-L ILI9488_Display:3.5_TFT_SPI_480_320 M1
+L Commander-Board-rescue:3.5_TFT_SPI_480_320-ILI9488_Display M1
 U 1 1 5F05872E
 P 13400 7550
